File: PCB/single valve board.brd (EAGLE design)
At the start: 25.4 x 38.1 mm, 6 parts, among them T1 2N2222

Commit message: board update
Connections:
- new net N$3: LED1.A, R1.2
- net GND: no longer LED1.K
- net N$2: now also LED1.K; no longer LED1.A, R1.2
Routing:
- net N$2: track 20.1 -> 8.04 mm
- net N$3: track 0.00 -> 10.1 mm
- net GND: track 10.8 -> 4.99 mm
Changed lines of the file:
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@@
 <wire x1="12.7" y1="1.905" x2="15.5575" y2="4.7625" width="0.254" layer="1" curve="-90"/>
 <wire x1="15.5575" y1="4.7625" x2="16.51" y2="4.7625" width="0.254" layer="1"/>
-<contactref element="LED1" pad="K"/>
-<wire x1="12.7" y1="1.905" x2="8.5725" y2="6.0325" width="0.254" layer="1"/>
 </signal>
 <signal name="5V">
@@
 <wire x1="19.685" y1="16.4465" x2="19.7739" y2="16.5354" width="0.254" layer="1" curve="-90"/>
 </signal>
+<signal name="N$3">
+<contactref element="R1" pad="2"/>
+<contactref element="LED1" pad="A"/>
+<wire x1="2.2579625" y1="16.509875" x2="8.5725" y2="8.5725" width="0.254" layer="1"/>
+</signal>
 <signal name="N$2">
-<contactref element="LED1" pad="A"/>
-<contactref element="R1" pad="2"/>
+<contactref element="LED1" pad="K"/>
 <contactref element="T1" pad="B"/>
-<wire x1="2.07686875" y1="12.52813125" x2="8.5725" y2="8.5725" width="0.254" layer="1"/>
-<wire x1="2.07686875" y1="12.52813125" x2="2.2579625" y2="16.509875" width="0.254" layer="1"/>
-<wire x1="8.5725" y1="8.5725" x2="9.8425" y2="7.3025" width="0.254" layer="1"/>
-<wire x1="9.8425" y1="7.3025" x2="16.51" y2="7.3025" width="0.254" layer="1"/>
+<wire x1="8.5725" y1="6.0325" x2="16.51" y2="7.3025" width="0.254" layer="1"/>
 </signal>
 </signals>

Commit message: pressure sensor board update
Parts:
- LED1: value (none) -> 2.2V 8mA
- renumbered T1 to SS8050
Changed lines of the file:
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@@
 </layers>
 <board>
-<fusionsync huburn="a.cGVyc29uYWw6dWUyYWM0Yzdl" projecturn="a.cGVyc29uYWw6dWUyYWM0YzdlIzIwMTgxMjA3MTY0NDE3NzU2" f3durn="urn:adsk.wipprod:dm.lineage:Ckdqxfa8RWO7gMxvI3SWJw" pcbguid="cf871d59-5326-4fd8-b094-b680d0f744d5" lastpulledtime="" lastsyncedchangeguid="3389f75c-7e19-a494-e700-5a38b7b5ce34"/>
+<fusionsync huburn="a.cGVyc29uYWw6dWUyYWM0Yzdl" projecturn="a.cGVyc29uYWw6dWUyYWM0YzdlIzIwMTgxMjA3MTY0NDE3NzU2" f3durn="urn:adsk.wipprod:dm.lineage:Ckdqxfa8RWO7gMxvI3SWJw" pcbguid="cf871d59-5326-4fd8-b094-b680d0f744d5" lastpulledtime="" lastsyncedchangeguid="c93bf3f4-3613-e115-6375-5f6b88c2930e"/>
 <plain>
 <wire x1="0" y1="0" x2="25.38" y2="0" width="0" layer="20"/>
@@
 <attribute name="VALUE" x="16.51" y="5.08" size="1.27" layer="27" rot="R180"/>
 </element>
-<element name="LED1" library="adafruit" library_urn="urn:adsk.eagle:library:420" package="LED5MM" package3d_urn="urn:adsk.eagle:package:6240538/1" value="" x="8.5725" y="7.3025" smashed="yes" rot="R270">
+<element name="LED1" library="adafruit" library_urn="urn:adsk.eagle:library:420" package="LED5MM" package3d_urn="urn:adsk.eagle:package:6240538/1" value="2.2V 8mA" x="8.5725" y="7.3025" smashed="yes" rot="R270">
 <attribute name="NAME" x="9.1059" y="4.1275" size="1.27" layer="25" ratio="10" rot="R270"/>
 <attribute name="VALUE" x="6.7691" y="4.1021" size="1.27" layer="27" ratio="10" rot="R270"/>
@@
 <attribute name="VALUE" x="2.8417" y="9.165015625" size="1.27" layer="27" ratio="10" rot="R89.6"/>
 </element>
-<element name="T1" library="adafruit" library_urn="urn:adsk.eagle:library:420" package="TO92-EBC-OVAL" package3d_urn="urn:adsk.eagle:package:6240647/1" value="2N2222" x="15.24" y="7.3025" smashed="yes" rot="R90">
+<element name="SS8050" library="adafruit" library_urn="urn:adsk.eagle:library:420" package="TO92-EBC-OVAL" package3d_urn="urn:adsk.eagle:package:6240647/1" value="2N2222" x="15.24" y="7.3025" smashed="yes" rot="R90">
 <attribute name="NAME" x="13.462" y="4.7625" size="1.27" layer="25" ratio="10" rot="R90"/>
 <attribute name="VALUE" x="19.812" y="4.7625" size="1.27" layer="27" ratio="10" rot="R90"/>
@@
 <signals>
 <signal name="N$1">
-<contactref element="T1" pad="C"/>
+<contactref element="SS8050" pad="C"/>
 <contactref element="SOLENOID1" pad="PAD11"/>
 <contactref element="D1" pad="A"/>
@@
 </signal>
 <signal name="GND">
-<contactref element="T1" pad="E"/>
+<contactref element="SS8050" pad="E"/>
 <contactref element="PINHEADER" pad="2"/>
 <wire x1="12.7" y1="1.905" x2="15.5575" y2="4.7625" width="0.254" layer="1" curve="-90"/>
@@
 <signal name="N$2">
 <contactref element="LED1" pad="K"/>
-<contactref element="T1" pad="B"/>
+<contactref element="SS8050" pad="B"/>
 <wire x1="8.5725" y1="6.0325" x2="16.51" y2="7.3025" width="0.254" layer="1"/>
 </signal>
