File: PCB/single valve board.sch (EAGLE design)
At the start: 6 parts, among them T1 2N2222

Commit message: pressure sensor board update
Parts:
- LED1: value (none) -> 2.2V 8mA
- renumbered T1 to SS8050
