File: PCB/3 valve front connect.sch (EAGLE design)
At the start: 17 parts, among them T1 2N2222, T2 2N2222, T3 2N2222

Commit message: board updates
Parts:
- removed JP1: (no value), adafruit:PINHD-1X3
- removed JP2: (no value), adafruit:PINHD-1X6
- added J1: (no value), SparkFun-Connectors:CONN_023.5MM
- added SV1: (no value), SparkFun-Connectors:CONN_04
- renumbered U$3 to VALVE3
Connections:
- removed net VALVEGPIO1: JP2.1, R1.1
- removed net VALVEGPIO2: JP2.2, R2.1
- removed net VALVEGPIO3: JP2.3, R3.1
- new net N$19: R3.1, SV1.1
- new net N$30: R1.1, SV1.3
- new net N$44: R2.1, SV1.2
- net 5V: now also J1.2; no longer JP1.1
- net GND: now also J1.1, SV1.4; no longer JP1.2, JP1.3, JP2.4
