File: PCB/pressure sensors.sch (EAGLE design)
At the start: 4 parts

Commit message: board updates
Parts:
- removed JP1: (no value), adafruit:PINHD-1X3
- added C3: 1µF, rcl:C-EU050-030X075
- added C4: 1nF, rcl:C-EU050-030X075
- added J1: (no value), SparkFun-Connectors:CONN_04
- added U$2: ADP5101, local eagle library:ADP5101
Connections:
- removed net N$1: C1.1, C2.1, JP1.2, U$1.P$1
- removed net N$2: C1.2, C2.2, JP1.1, U$1.P$6
- new net 5V: C1.1, C2.1, C3.1, C4.1, J1.2, U$1.P$1, U$2.P$1
- new net GND: C1.2, C2.2, C3.2, C4.2, J1.1, U$1.P$6, U$2.P$6
- new net N$6: J1.4, U$2.P$3
- net N$3: now also J1.3; no longer JP1.3
Changed lines of the file:
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@@
 <layer number="112" name="tSilk" color="7" fill="1" visible="no" active="yes"/>
 <layer number="113" name="ReferenceLS" color="7" fill="1" visible="no" active="no"/>
+<layer number="114" name="Badge_Outline" color="7" fill="1" visible="yes" active="yes"/>
+<layer number="115" name="ReferenceISLANDS" color="7" fill="1" visible="yes" active="yes"/>
 <layer number="116" name="Patch_BOT" color="9" fill="4" visible="no" active="yes"/>
 <layer number="118" name="Rect_Pads" color="7" fill="1" visible="no" active="no"/>
@@
 <part name="C1" library="rcl" library_urn="urn:adsk.eagle:library:334" deviceset="C-EU" device="050-030X075" package3d_urn="urn:adsk.eagle:package:23640/1" value="1µF"/>
 <part name="C2" library="rcl" library_urn="urn:adsk.eagle:library:334" deviceset="C-EU" device="050-030X075" package3d_urn="urn:adsk.eagle:package:23640/1" value="1nF"/>
-<part name="JP1" library="adafruit" library_urn="urn:adsk.eagle:library:420" deviceset="PINHD-1X3" device="" package3d_urn="urn:adsk.eagle:package:6240710/1"/>
+<part name="U$2" library="local eagle library" deviceset="ADP5101" device="" package3d_urn="urn:adsk.eagle:package:7362871/1"/>
+<part name="C3" library="rcl" library_urn="urn:adsk.eagle:library:334" deviceset="C-EU" device="050-030X075" package3d_urn="urn:adsk.eagle:package:23640/1" value="1µF"/>
+<part name="C4" library="rcl" library_urn="urn:adsk.eagle:library:334" deviceset="C-EU" device="050-030X075" package3d_urn="urn:adsk.eagle:package:23640/1" value="1nF"/>
+<part name="J1" library="SparkFun-Connectors" library_urn="urn:adsk.eagle:library:513" deviceset="CONN_04" device="" package3d_urn="urn:adsk.eagle:package:38085/1"/>
 </parts>
 <sheets>
@@
 <attribute name="VALUE" x="21.844" y="56.261" size="1.778" layer="96"/>
 </instance>
-<instance part="JP1" gate="A" x="-2.54" y="86.36" smashed="yes">
-<attribute name="NAME" x="-8.89" y="92.075" size="1.778" layer="95"/>
-<attribute name="VALUE" x="-8.89" y="78.74" size="1.778" layer="96"/>
+<instance part="U$2" gate="G$1" x="106.68" y="58.42" smashed="yes"/>
+<instance part="C3" gate="G$1" x="93.98" y="60.96" smashed="yes">
+<attribute name="NAME" x="95.504" y="61.341" size="1.778" layer="95"/>
+<attribute name="VALUE" x="95.504" y="56.261" size="1.778" layer="96"/>
+</instance>
+<instance part="C4" gate="G$1" x="81.28" y="60.96" smashed="yes">
+<attribute name="NAME" x="82.804" y="61.341" size="1.778" layer="95"/>
+<attribute name="VALUE" x="82.804" y="56.261" size="1.778" layer="96"/>
+</instance>
+<instance part="J1" gate="G$1" x="-15.24" y="86.36" smashed="yes">
+<attribute name="VALUE" x="-20.32" y="78.994" size="1.778" layer="96" font="vector"/>
+<attribute name="NAME" x="-20.32" y="94.488" size="1.778" layer="95" font="vector"/>
 </instance>
 </instances>
@@
 </busses>
 <nets>
-<net name="N$1" class="0">
+<net name="5V" class="0">
 <segment>
 <pinref part="C2" gate="G$1" pin="1"/>
@@
 <wire x1="33.02" y1="68.58" x2="45.72" y2="68.58" width="0.1524" layer="91"/>
 <wire x1="45.72" y1="68.58" x2="45.72" y2="63.5" width="0.1524" layer="91"/>
-<pinref part="JP1" gate="A" pin="2"/>
-<wire x1="-5.08" y1="86.36" x2="5.08" y2="86.36" width="0.1524" layer="91"/>
-<wire x1="5.08" y1="86.36" x2="5.08" y2="63.5" width="0.1524" layer="91"/>
+<pinref part="C4" gate="G$1" pin="1"/>
+<pinref part="C3" gate="G$1" pin="1"/>
+<wire x1="5.08" y1="76.2" x2="5.08" y2="63.5" width="0.1524" layer="91"/>
+<wire x1="81.28" y1="63.5" x2="93.98" y2="63.5" width="0.1524" layer="91"/>
+<junction x="81.28" y="63.5"/>
+<wire x1="93.98" y1="63.5" x2="93.98" y2="68.58" width="0.1524" layer="91"/>
+<junction x="93.98" y="63.5"/>
+<pinref part="U$2" gate="G$1" pin="P$1"/>
+<wire x1="93.98" y1="68.58" x2="106.68" y2="68.58" width="0.1524" layer="91"/>
+<wire x1="106.68" y1="68.58" x2="106.68" y2="63.5" width="0.1524" layer="91"/>
+<wire x1="63.5" y1="63.5" x2="81.28" y2="63.5" width="0.1524" layer="91"/>
+<wire x1="0" y1="86.36" x2="5.08" y2="76.2" width="0.1524" layer="91"/>
+<wire x1="5.08" y1="76.2" x2="63.5" y2="76.2" width="0.1524" layer="91"/>
+<wire x1="63.5" y1="76.2" x2="63.5" y2="63.5" width="0.1524" layer="91"/>
+<pinref part="J1" gate="G$1" pin="2"/>
+<wire x1="0" y1="86.36" x2="-10.16" y2="86.36" width="0.1524" layer="91"/>
 </segment>
 </net>
-<net name="N$2" class="0">
+<net name="GND" class="0">
 <segment>
 <pinref part="C2" gate="G$1" pin="2"/>
-<wire x1="-2.54" y1="55.88" x2="20.32" y2="55.88" width="0.1524" layer="91"/>
+<wire x1="-2.54" y1="55.88" x2="5.08" y2="55.88" width="0.1524" layer="91"/>
 <pinref part="C1" gate="G$1" pin="2"/>
+<wire x1="5.08" y1="55.88" x2="20.32" y2="55.88" width="0.1524" layer="91"/>
 <wire x1="20.32" y1="55.88" x2="33.02" y2="55.88" width="0.1524" layer="91"/>
 <junction x="20.32" y="55.88"/>
@@
 <wire x1="33.02" y1="53.34" x2="45.72" y2="53.34" width="0.1524" layer="91"/>
 <junction x="33.02" y="55.88"/>
-<pinref part="JP1" gate="A" pin="1"/>
-<wire x1="-5.08" y1="88.9" x2="-2.54" y2="88.9" width="0.1524" layer="91"/>
-<wire x1="-2.54" y1="88.9" x2="-2.54" y2="55.88" width="0.1524" layer="91"/>
+<wire x1="-10.16" y1="83.82" x2="-2.54" y2="55.88" width="0.1524" layer="91"/>
+<wire x1="5.08" y1="55.88" x2="5.08" y2="43.18" width="0.1524" layer="91"/>
+<wire x1="5.08" y1="43.18" x2="2.54" y2="43.18" width="0.1524" layer="91"/>
+<junction x="5.08" y="55.88"/>
+<pinref part="C4" gate="G$1" pin="2"/>
+<wire x1="58.42" y1="55.88" x2="73.66" y2="55.88" width="0.1524" layer="91"/>
+<pinref part="C3" gate="G$1" pin="2"/>
+<wire x1="73.66" y1="55.88" x2="81.28" y2="55.88" width="0.1524" layer="91"/>
+<wire x1="81.28" y1="55.88" x2="93.98" y2="55.88" width="0.1524" layer="91"/>
+<junction x="81.28" y="55.88"/>
+<pinref part="U$2" gate="G$1" pin="P$6"/>
+<wire x1="93.98" y1="55.88" x2="93.98" y2="53.34" width="0.1524" layer="91"/>
+<wire x1="93.98" y1="53.34" x2="106.68" y2="53.34" width="0.1524" layer="91"/>
+<junction x="93.98" y="55.88"/>
+<wire x1="5.08" y1="43.18" x2="73.66" y2="43.18" width="0.1524" layer="91"/>
+<wire x1="73.66" y1="43.18" x2="73.66" y2="55.88" width="0.1524" layer="91"/>
+<junction x="73.66" y="55.88"/>
+<pinref part="J1" gate="G$1" pin="1"/>
 </segment>
 </net>
@@
 <segment>
 <pinref part="U$1" gate="G$1" pin="P$3"/>
-<pinref part="JP1" gate="A" pin="3"/>
-<wire x1="50.8" y1="63.5" x2="50.8" y2="83.82" width="0.1524" layer="91"/>
-<wire x1="50.8" y1="83.82" x2="-5.08" y2="83.82" width="0.1524" layer="91"/>
+<wire x1="50.8" y1="63.5" x2="50.8" y2="88.9" width="0.1524" layer="91"/>
+<pinref part="J1" gate="G$1" pin="3"/>
+<wire x1="-10.16" y1="88.9" x2="50.8" y2="88.9" width="0.1524" layer="91"/>
 </segment>
 </net>
+<net name="N$6" class="0">
+<segment>
+<pinref part="U$2" gate="G$1" pin="P$3"/>
+<wire x1="111.76" y1="63.5" x2="111.76" y2="91.44" width="0.1524" layer="91"/>
+<pinref part="J1" gate="G$1" pin="4"/>
+<wire x1="-10.16" y1="91.44" x2="111.76" y2="91.44" width="0.1524" layer="91"/>
+</segment>
+</net>
