File: PCB/4 valve front connect.sch (EAGLE design)
At the start: 17 parts, among them T1 2N2222, T2 2N2222, T3 2N2222

Commit message: 4 valve boards
Parts:
- removed JP1: (no value), adafruit:PINHD-1X3
- removed JP2: (no value), adafruit:PINHD-1X6
- added D4: 1N4004, adafruit:1N4004
- added J1: (no value), SparkFun-Connectors:CONN_023.5MM
- added J2: (no value), SparkFun-Connectors:CONN_02
- added LED4: (no value), adafruit:LED5MM
- added R4: (no value), adafruit:R-US_0207/10
- added SV1: (no value), SparkFun-Connectors:CONN_05
- added T4: 2N2222, adafruit:2N2222
- added VALVE3: (no value), local eagle library:VALVE
Connections:
- removed net VALVEGPIO1: JP2.1, R1.1
- removed net VALVEGPIO2: JP2.2, R2.1
- removed net VALVEGPIO3: JP2.3, R3.1
- new net N$12: LED4.A, R4.2
- new net N$13: R4.1, SV1.1
- new net N$14: R2.1, SV1.3
- new net N$19: R3.1, SV1.2
- new net N$30: R1.1, SV1.4
- new net N$4: D4.A, T4.C, U$3.PINS2
- new net N$8: LED4.C, T4.B
- net 5V: now also D4.C, J1.2, J2.2, VALVE3.PINS1; no longer JP1.1
- net GND: now also J1.1, J2.1, SV1.5, T4.E; no longer JP1.2, JP1.3, JP2.4
- net N$9: now also VALVE3.PINS2; no longer U$3.PINS2
