File: PCB/8 valve.sch (EAGLE design)
At the start: 17 parts, among them T1 2N2222, T2 2N2222, T3 2N2222

Commit message: 4 valve boards
Parts:
- removed JP1: (no value), adafruit:PINHD-1X3
- removed JP2: (no value), adafruit:PINHD-1X6
- added D10, D11, D12, D4, D9: 1N4004, adafruit:1N4004
- added J1: (no value), SparkFun-Connectors:CONN_023.5MM
- added LED10, LED11, LED12, LED4, LED9: (no value), adafruit:LED5MM
- added R10, R11, R12, R4, R9: (no value), adafruit:R-US_0207/10
- added SV1: (no value), SparkFun-Connectors:CONN_09
- added SV3: (no value), SparkFun-Connectors:CONN_05
- added T10, T11, T12, T4, T9: 2N2222, adafruit:2N2222
- added U$7, U$8, U$9, VALVE2, VALVE3: (no value), local eagle library:VALVE
Connections:
- removed net VALVEGPIO1: JP2.1, R1.1
- removed net VALVEGPIO2: JP2.2, R2.1
- removed net VALVEGPIO3: JP2.3, R3.1
- new net N$12: LED4.A, R4.2
- new net N$13: R4.1, SV1.1
- new net N$14: R2.1, SV1.3
- new net N$15: R12.1, SV3.1
- new net N$19: R3.1, SV1.2
- new net N$23: R9.1, SV1.6
- new net N$30: R1.1, SV1.4
- new net N$37: D9.A, T9.C, U$7.PINS2
- new net N$38: LED9.C, T9.B
- new net N$39: LED9.A, R9.2
- new net N$4: D4.A, T4.C, U$3.PINS2
- new net N$41: D10.A, T10.C, U$8.PINS2
- new net N$43: LED10.C, T10.B
- new net N$44: LED10.A, R10.2
- new net N$45: D11.A, T11.C, VALVE2.PINS2
- new net N$46: LED11.C, T11.B
- new net N$47: LED11.A, R11.2
- new net N$49: R11.1, SV3.2
- new net N$53: D12.A, T12.C, U$9.PINS2
- new net N$54: LED12.C, T12.B
- new net N$55: LED12.A, R12.2
- new net N$57: R10.1
- new net N$8: LED4.C, T4.B
- net 5V: now also D10.C, D11.C, D12.C, D4.C, D9.C, J1.2, U$7.PINS1, U$8.PINS1, U$9.PINS1, VALVE2.PINS1, VALVE3.PINS1; no longer JP1.1
- net GND: now also J1.1, SV1.5, SV3.5, T10.E, T11.E, T12.E, T4.E, T9.E; no longer JP1.2, JP1.3, JP2.4
- net N$9: now also VALVE3.PINS2; no longer U$3.PINS2
