File: PCB/mini system.brd (EAGLE design)
At the start: 126.7 x 88.9 mm, 24 parts, among them T1 2N2222, T2 2N2222, T3 2N2222

Commit message: new board
Other:
- board size 126.7 x 88.9 mm -> 127 x 79.4 mm
Changed lines of the file:
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@@
 <board>
 <plain>
-<wire x1="0" y1="85.715" x2="0" y2="3.175" width="0" layer="20"/>
-<wire x1="0" y1="3.175" x2="3.175" y2="0" width="0" layer="20" curve="90"/>
-<wire x1="3.175" y1="0" x2="123.495" y2="0" width="0" layer="20"/>
-<wire x1="123.495" y1="0" x2="126.67" y2="3.175" width="0" layer="20" curve="90"/>
-<wire x1="126.67" y1="3.175" x2="126.67" y2="85.715" width="0" layer="20"/>
-<wire x1="126.67" y1="85.715" x2="123.495" y2="88.89" width="0" layer="20" curve="90"/>
+<wire x1="0" y1="85.715" x2="0" y2="12.7" width="0" layer="20"/>
+<wire x1="0" y1="12.7" x2="3.175" y2="9.525" width="0" layer="20" curve="90"/>
+<wire x1="3.175" y1="9.525" x2="123.8125" y2="9.525" width="0" layer="20"/>
+<wire x1="123.8125" y1="9.525" x2="126.9875" y2="12.7" width="0" layer="20" curve="90"/>
+<wire x1="126.9875" y1="12.7" x2="126.9875" y2="85.715" width="0" layer="20"/>
+<wire x1="126.9875" y1="85.715" x2="123.495" y2="88.89" width="0" layer="20" curve="90"/>
 <wire x1="123.495" y1="88.89" x2="3.175" y2="88.89" width="0" layer="20"/>
 <wire x1="3.175" y1="88.89" x2="0" y2="85.715" width="0" layer="20" curve="90"/>
 <hole x="3.175" y="85.725" drill="3.175"/>
-<hole x="3.175" y="3.175" drill="3.175"/>
-<hole x="123.825" y="3.175" drill="3.175"/>
+<hole x="3.175" y="12.7" drill="3.175"/>
+<hole x="123.825" y="12.7" drill="3.175"/>
 <hole x="123.825" y="85.725" drill="3.175"/>
 </plain>
@@
 <contactref element="R3" pad="1"/>
 <contactref element="U$1" pad="D3"/>
-<wire x1="58.42" y1="69.85" x2="58.42" y2="66.04" width="0.254" layer="16"/>
+<wire x1="58.42" y1="69.85" x2="58.42" y2="66.04" width="0.381" layer="16"/>
 </signal>
 <signal name="N$7">
@@
 <contactref element="U$1" pad="D2"/>
 <wire x1="55.88" y1="69.85" x2="55.88" y2="68.58" width="0.254" layer="16"/>
-<wire x1="55.88" y1="68.58" x2="53.34" y2="66.04" width="0.254" layer="16" curve="-90"/>
+<wire x1="55.88" y1="68.58" x2="53.34" y2="66.04" width="0.381" layer="16" curve="-90"/>
 </signal>
 <signal name="N$4">
@@
 <contactref element="U$1" pad="D4"/>
 <wire x1="60.96" y1="69.85" x2="60.96" y2="68.58" width="0.254" layer="16"/>
-<wire x1="60.96" y1="68.58" x2="63.5" y2="66.04" width="0.254" layer="16" curve="90"/>
+<wire x1="60.96" y1="68.58" x2="63.5" y2="66.04" width="0.381" layer="16" curve="90"/>
 </signal>
 <signal name="5V">
