File: PCB/mini system- 5 components vertical moved nano.brd (EAGLE design)
At the start: 127 x 101.6 mm, 33 parts, among them J2 POWER_JACK, T1 2N2222, T2 2N2222, T3 2N2222, T4 2N2222, T5 2N2222

Commit message: 2
Parts:
- added C5: (no value), adafruit:E2,5-7
- moved C4 3.68 mm to (36.1, 88.8)
- moved R2 2.67 mm to (104.3, 53.3)
- moved T2 2.67 mm to (96.1, 53.3)
- moved R1 1.78 mm to (104.3, 33.8)
- moved R7 1.78 mm to (104.3, 43.6)
- moved T1 1.78 mm to (96.1, 33.8)
- moved T4 1.78 mm to (96.1, 43.6)
- moved S2 0.59 mm to (98.1, 5.33)
- moved S3 0.30 mm to (88.1, 5.33)
- moved R3 0.13 mm to (104.3, 24.0)
- moved R8 0.13 mm to (104.3, 63.1)
Connections:
- net 5V: now also C5.+
- net GND: now also C5.-
Routing:
- net 5V: track 393.9 -> 411.5 mm
- net GND: track 382.2 -> 385.7 mm
- net N$5: track 29.2 -> 27.0 mm
- net N$7: track 41.7 -> 39.7 mm
- net N$18: track 50.6 -> 49.5 mm
- net N$4: track 60.4 -> 59.3 mm
- net N$8: track 110.6 -> 109.9 mm
- net N$16: track 92.3 -> 93.0 mm
- net N$28: track 88.4 -> 89.0 mm
